File: hardware/smartPlug-PCB/smartPlug-PCB.kicad_pcb (KiCad board)
At the start: 2 copper layers, 90 x 55 mm, 10 parts, among them J1 Screw_Terminal_01x02, J2 Screw_Terminal_01x02, K1 SRD-05VDC-SL-C, Q1 2N3904, SW2 SW_Push, U1 ESP32-C3_SUPERMINI_TH, U2 HLK-PM01

Commit message: Added M3 scre holes to PCB
Parts:
- added REF**: MountingHole_3.2mm_M3, MountingHole:MountingHole_3.2mm_M3, F.Cu at (74.5, 100.0)
- added REF**: MountingHole_3.2mm_M3, MountingHole:MountingHole_3.2mm_M3, F.Cu at (156.0, 100.0)
- added REF**: MountingHole_3.2mm_M3, MountingHole:MountingHole_3.2mm_M3, F.Cu at (74.5, 38.5)
- added REF**: MountingHole_3.2mm_M3, MountingHole:MountingHole_3.2mm_M3, F.Cu at (156.5, 38.5)
Other:
- board size 90 x 55 mm -> 91 x 71.5 mm
